File: hw.brd (EAGLE design)
At the start: 64.8 x 81.3 mm, 37 parts, among them IC1 MIC_I2S_SPH0645, Q3 DMG3415U, U1 MAX98357A, U2 AP2112-3.3, U3 MCP73831T-2ACI/OT, X2 JSTPH

Commit message: ground plane!
Routing:
- net GND: track 22.6 -> 32.7 mm
- added copper zone on layer 16, net GND
Changed lines of the file:
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@@
 <wire x1="27.94" y1="53.34" x2="19.05" y2="53.34" width="0.254" layer="16"/>
 <wire x1="27.94" y1="73.66" x2="19.05" y2="73.66" width="0.254" layer="16"/>
-<wire x1="27.94" y1="73.66" x2="58.42" y2="76.2" width="0" layer="19" extent="1-1"/>
-<wire x1="27.94" y1="53.34" x2="27.94" y2="73.66" width="0" layer="19" extent="1-1"/>
-<wire x1="33.87" y1="33.02" x2="27.94" y2="53.34" width="0" layer="19" extent="16-16"/>
-<wire x1="32.46" y1="30.48" x2="33.87" y2="33.02" width="0" layer="19" extent="16-16"/>
-<wire x1="33.02" y1="25.72" x2="32.46" y2="30.48" width="0" layer="19" extent="16-16"/>
-<wire x1="30.48" y1="25.72" x2="33.02" y2="25.72" width="0" layer="19" extent="16-16"/>
-<wire x1="36.83" y1="27.94" x2="33.02" y2="25.72" width="0" layer="19" extent="16-16"/>
-<wire x1="32" y1="18.01" x2="33.02" y2="25.72" width="0" layer="19" extent="16-16"/>
-<wire x1="36.83" y1="16.51" x2="33.25" y2="16.26" width="0" layer="19" extent="16-16"/>
-<wire x1="26.35" y1="17.78" x2="30.25" y2="16.76" width="0" layer="19" extent="16-16"/>
-<wire x1="26.35" y1="15.24" x2="26.35" y2="17.78" width="0" layer="19" extent="16-16"/>
-<wire x1="32.7" y1="10.16" x2="33.25" y2="16.26" width="0" layer="19" extent="16-16"/>
-<wire x1="32.7" y1="7.62" x2="32.7" y2="10.16" width="0" layer="19" extent="16-16"/>
-<wire x1="49.96" y1="39.38" x2="33.87" y2="33.02" width="0" layer="19" extent="16-16"/>
-<wire x1="55.88" y1="33.97" x2="49.96" y2="39.38" width="0" layer="19" extent="16-16"/>
-<wire x1="60.9299" y1="33.02" x2="55.88" y2="33.97" width="0" layer="19" extent="16-16"/>
-<wire x1="63.5" y1="28.79" x2="60.9299" y2="33.02" width="0" layer="19" extent="16-16"/>
-<wire x1="66.04" y1="28.79" x2="63.5" y2="28.79" width="0" layer="19" extent="16-16"/>
-<wire x1="66.89" y1="31.75" x2="66.04" y2="28.79" width="0" layer="19" extent="16-16"/>
-<wire x1="66.99" y1="34.29" x2="66.89" y2="31.75" width="0" layer="19" extent="16-16"/>
-<wire x1="66.99" y1="36.83" x2="66.99" y2="34.29" width="0" layer="19" extent="16-16"/>
-<wire x1="62.23" y1="21.5599" x2="63.5" y2="28.79" width="0" layer="19" extent="16-16"/>
-<wire x1="63.18" y1="19.05" x2="62.23" y2="21.5599" width="0" layer="19" extent="16-16"/>
-<wire x1="61.23" y1="13.86" x2="63.18" y2="19.05" width="0" layer="19" extent="16-16"/>
+<polygon width="0.254" layer="16">
+<vertex x="15.24" y="81.28"/>
+<vertex x="80.01" y="81.28"/>
+<vertex x="80.01" y="0"/>
+<vertex x="15.24" y="0"/>
+</polygon>
+<wire x1="34.29" y1="19.05" x2="31.75" y2="19.05" width="0.254" layer="16"/>
+<wire x1="31.75" y1="19.05" x2="31.75" y2="18.8417125" width="0.254" layer="16"/>
+<wire x1="31.75" y1="18.8417125" x2="31.9318" y2="18.6599125" width="0.254" layer="16"/>
+<wire x1="31.9318" y1="18.6599125" x2="31.9318" y2="17.9418" width="0.254" layer="16"/>
+<wire x1="36.83" y1="16.51" x2="34.29" y2="19.05" width="0.254" layer="16"/>
+<wire x1="31.75" y1="16.51" x2="32.258" y2="16.002" width="0.254" layer="16"/>
+<wire x1="32.258" y1="16.002" x2="32.258" y2="13.97" width="0.254" layer="16"/>
 </signal>
 <signal name="SD_MODE">

Commit message: changing cherrymx part to avoid large etch-off area
Parts:
- removed S1, S2: CHERRY_MX, cherry:CHERRY_MX
- added U$16, U$20: CHERRY-MX, cherrymx:CHERRY-MX
Connections:
- net BTN1: now also U$20.SW2; no longer S2.S2
- net BTN2: now also U$16.SW2; no longer S1.S2
- net GND: now also U$16.SW1, U$20.SW1; no longer S1.S1, S2.S1
Routing:
- net GND: track 32.7 -> 14.9 mm
- net BTN2: track 56.7 -> 56.2 mm
Changed lines of the file:
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@@
 <attribute name="VALUE" x="73.66" y="71.12" size="1.27" layer="27" font="vector" align="bottom-right"/>
-</element>
-<element name="S1" library="cherry" package="CHERRY_MX" value="CHERRY_MX" x="31.75" y="71.12" smashed="yes">
-<attribute name="FARNELL" value="2292961" x="31.75" y="71.12" size="1.778" layer="27" display="off"/>
-<attribute name="MOUSER" value="540-MX1A-11NW" x="31.75" y="71.12" size="1.778" layer="27" display="off"/>
-<attribute name="NAME" x="24.13" y="80.01" size="1.27" layer="25"/>
-<attribute name="VALUE" x="36.83" y="34.29" size="1.27" layer="25"/>
-</element>
-<element name="S2" library="cherry" package="CHERRY_MX" value="CHERRY_MX" x="31.75" y="50.8" smashed="yes">
-<attribute name="FARNELL" value="2292961" x="31.75" y="50.8" size="1.778" layer="27" display="off"/>
-<attribute name="MOUSER" value="540-MX1A-11NW" x="31.75" y="50.8" size="1.778" layer="27" display="off"/>
-<attribute name="NAME" x="24.13" y="59.69" size="1.27" layer="25"/>
-<attribute name="VALUE" x="21.59" y="-2.54" size="1.27" layer="25" rot="R270"/>
 </element>
 <element name="U1" library="microbuilder" package="QFN16_3MM" value="MAX98357A" x="31.75" y="16.51" smashed="yes" rot="MR0">
@@
 <attribute name="VALUE" x="33.655" y="20.32" size="0.4064" layer="27" ratio="10" rot="R270"/>
 </element>
+<element name="U$16" library="cherrymx" package="CHERRY-MX" value="CHERRY-MX" x="31.75" y="69.85" smashed="yes"/>
+<element name="U$20" library="cherrymx" package="CHERRY-MX" value="CHERRY-MX" x="31.75" y="50.8" smashed="yes"/>
 </elements>
 <signals>
@@
 <contactref element="JP2" pad="2"/>
 <contactref element="JP1" pad="2"/>
-<contactref element="S2" pad="S1"/>
-<contactref element="S1" pad="S1"/>
 <contactref element="U$12" pad="2"/>
 <wire x1="30.25" y1="16.76" x2="30.3182" y2="16.6918" width="0.254" layer="16"/>
@@
 <wire x1="31.75" y1="17.32486875" x2="31.9318" y2="17.50666875" width="0.254" layer="16"/>
 <wire x1="31.9318" y1="17.50666875" x2="31.9318" y2="17.9418" width="0.254" layer="16"/>
-<wire x1="27.94" y1="53.34" x2="19.05" y2="53.34" width="0.254" layer="16"/>
-<wire x1="27.94" y1="73.66" x2="19.05" y2="73.66" width="0.254" layer="16"/>
 <polygon width="0.254" layer="16">
 <vertex x="15.24" y="81.28"/>
@@
 <wire x1="31.75" y1="16.51" x2="32.258" y2="16.002" width="0.254" layer="16"/>
 <wire x1="32.258" y1="16.002" x2="32.258" y2="13.97" width="0.254" layer="16"/>
+<contactref element="U$20" pad="SW1"/>
+<contactref element="U$16" pad="SW1"/>
 </signal>
 <signal name="SD_MODE">
@@
 </signal>
 <signal name="BTN1">
-<contactref element="S2" pad="S2"/>
 <contactref element="U$12" pad="27"/>
-<wire x1="74.73" y1="34.3" x2="53.15" y2="55.88" width="0.3048" layer="16"/>
-<wire x1="53.15" y1="55.88" x2="34.29" y2="55.88" width="0.3048" layer="16"/>
+<contactref element="U$20" pad="SW2"/>
+<wire x1="67.73625" y1="37.8848" x2="67.5252" y2="37.8848" width="0.3048" layer="16"/>
+<wire x1="67.5252" y1="37.8848" x2="49.53" y2="55.88" width="0.3048" layer="16"/>
+<wire x1="74.73" y1="34.3" x2="71.32105" y2="34.3" width="0.3048" layer="16"/>
+<wire x1="71.32105" y1="34.3" x2="67.73625" y2="37.8848" width="0.3048" layer="16"/>
+<wire x1="49.53" y1="55.88" x2="34.29" y2="55.88" width="0.3048" layer="16"/>
 </signal>
 <signal name="BTN2">
-<contactref element="S1" pad="S2"/>
 <contactref element="U$12" pad="28"/>
-<wire x1="74.73" y1="36.84" x2="35.37" y2="76.2" width="0.3048" layer="16"/>
-<wire x1="35.37" y1="76.2" x2="34.29" y2="76.2" width="0.3048" layer="16"/>
+<contactref element="U$16" pad="SW2"/>
+<wire x1="74.73" y1="36.84" x2="36.64" y2="74.93" width="0.3048" layer="16"/>
+<wire x1="36.64" y1="74.93" x2="34.29" y2="74.93" width="0.3048" layer="16"/>
 </signal>
 <signal name="VDD">
